File: 5V_8A.sch (KiCad schematic (older format))
At the start: 14 parts, among them Q2 CSD18503Q5A, U2 RT7258GQW

Commit message: More PCB tweaks
Parts:
- C14: value C-0603 -> 1u; BOM CAP MLCC 100pF C0G 50V 5% [0603] -> CAP MLCC 1u ≥X5R 16V 20% [0603]
- R5: value R-0603 -> 1k; BOM RES SMD 1k 5% [0603] -> RES SMD 1k 1% [0603]
- R6: value R-0603 -> 95k3; BOM RES SMD 1k 5% [0603] -> RES SMD 95k3 1% [0603]
- R7: value R-0603 -> 18k; BOM RES SMD 1k 5% [0603] -> RES SMD 18k 1% [0603]
- R8: value R-0603 -> 100; BOM RES SMD 1k 5% [0603] -> RES SMD 100 1% [0603]
Other:
- note added: "0.808V"
- note added: "5.09V with sense\n5.14V floating sense"
Changed lines of the file:
@@
 encoding utf-8
 Sheet 3 7
-Title ""
-Date ""
-Rev ""
-Comp ""
-Comment1 ""
+Title "5V 8A regulator block"
+Date "2016-07-01"
+Rev "R1"
+Comp "c4757p / semianalog"
+Comment1 "C4-0 POWER SUPPLY"
 Comment2 ""
 Comment3 ""
@@
 AR Path="/577479AE/57749C02" Ref="R1"  Part="1"
 F 0 "R1" H 7163 3946 50  0000 L CNN
-F 1 "R-0603" H 7163 3855 50  0000 L CNN
+F 1 "1k" H 7163 3855 50  0000 L CNN
 F 2 "IPC7351-Nominal:RESC1608X50" H 7100 3900 50  0001 C CNN
 F 3 "" H 7100 3950 60  0000 C CNN
-F 4 "RES SMD 1k 5% [0603]" H 7850 4450 60  0001 C CNN "BOM"
+F 4 "RES SMD 1k 1% [0603]" H 7850 4450 60  0001 C CNN "BOM"
 	1    7100 3900
 	1    0    0    -1
@@
 AR Path="/577479AE/57749C62" Ref="R2"  Part="1"
 F 0 "R2" H 7163 4346 50  0000 L CNN
-F 1 "R-0603" H 7163 4255 50  0000 L CNN
+F 1 "95k3" H 7163 4255 50  0000 L CNN
 F 2 "IPC7351-Nominal:RESC1608X50" H 7100 4300 50  0001 C CNN
 F 3 "" H 7100 4350 60  0000 C CNN
-F 4 "RES SMD 1k 5% [0603]" H 7850 4850 60  0001 C CNN "BOM"
+F 4 "RES SMD 95k3 1% [0603]" H 7850 4850 60  0001 C CNN "BOM"
 	1    7100 4300
 	1    0    0    -1
@@
 AR Path="/577479AE/57749CA9" Ref="R3"  Part="1"
 F 0 "R3" H 7163 4746 50  0000 L CNN
-F 1 "R-0603" H 7163 4655 50  0000 L CNN
+F 1 "18k" H 7163 4655 50  0000 L CNN
 F 2 "IPC7351-Nominal:RESC1608X50" H 7100 4700 50  0001 C CNN
 F 3 "" H 7100 4750 60  0000 C CNN
-F 4 "RES SMD 1k 5% [0603]" H 7850 5250 60  0001 C CNN "BOM"
+F 4 "RES SMD 18k 1% [0603]" H 7850 5250 60  0001 C CNN "BOM"
 	1    7100 4700
-	1    0    0    -1
-$EndComp
-$Comp
-L C-0603 C14
-U 1 1 57749CE4
-P 7600 3900
-AR Path="/577485D6/57749CE4" Ref="C14"  Part="1"
-AR Path="/577479AE/57749CE4" Ref="C7"  Part="1"
-F 0 "C7" H 7713 3946 50  0000 L CNN
-F 1 "C-0603" H 7713 3855 50  0000 L CNN
-F 2 "IPC7351-Nominal:CAPC1608X55" H 7600 3900 50  0001 C CNN
-F 3 "" H 7590 3875 60  0000 C CNN
-F 4 "CAP MLCC 100pF C0G 50V 5% [0603]" H 8400 4450 60  0001 C CNN "BOM"
-	1    7600 3900
 	1    0    0    -1
 $EndComp
@@
 AR Path="/577479AE/57749E45" Ref="R4"  Part="1"
 F 0 "R4" V 8050 4100 50  0000 C CNN
-F 1 "R-0603" V 8141 4100 50  0000 C CNN
+F 1 "100" V 8141 4100 50  0000 C CNN
 F 2 "IPC7351-Nominal:RESC1608X50" H 8250 4100 50  0001 C CNN
 F 3 "" H 8250 4150 60  0000 C CNN
-F 4 "RES SMD 1k 5% [0603]" H 9000 4650 60  0001 C CNN "BOM"
+F 4 "RES SMD 100 1% [0603]" H 9000 4650 60  0001 C CNN "BOM"
 	1    8250 4100
 	0    1    1    0
@@
 IN
 Connection ~ 3250 3200
+$Comp
+L C-0603 C14
+U 1 1 57749CE4
+P 7600 3900
+AR Path="/577485D6/57749CE4" Ref="C14"  Part="1"
+AR Path="/577479AE/57749CE4" Ref="C7"  Part="1"
+F 0 "C7" H 7713 3946 50  0000 L CNN
+F 1 "1u" H 7713 3855 50  0000 L CNN
+F 2 "IPC7351-Nominal:CAPC1608X55" H 7600 3900 50  0001 C CNN
+F 3 "" H 7590 3875 60  0000 C CNN
+F 4 "CAP MLCC 1u ≥X5R 16V 20% [0603]" H 8400 4450 60  0001 C CNN "BOM"
+	1    7600 3900
+	1    0    0    -1
+$EndComp
+Text Notes 6600 4450 0    60   ~ 0
+0.808V
+Text Notes 7750 3600 0    60   ~ 0
+5.09V with sense\n5.14V floating sense
 $EndSCHEMATC
