File: Supervisor.sch (KiCad schematic (older format))
At the start: 10 parts, among them J2 PDI, U7 ATXMEGA32E5-MU, U8 MCP1754ST-3302E/CB

Commit message: More PCB tweaks
Changed lines of the file:
@@
 encoding utf-8
 Sheet 7 7
-Title ""
-Date ""
-Rev ""
-Comp ""
-Comment1 ""
+Title "Supervisor"
+Date "2016-07-01"
+Rev "R1"
+Comp "c4757p / semianalog"
+Comment1 "C4-0 POWER SUPPLY"
 Comment2 ""
 Comment3 ""
@@
 $EndComp
 Wire Wire Line
-	1700 2200 1900 2200
-Wire Wire Line
-	1900 2200 2300 2200
+	1700 2200 2300 2200
 Wire Wire Line
 	1900 2300 1900 2200
@@
 	1900 2600 1900 2500
 Wire Wire Line
-	3000 2200 3300 2200
-Wire Wire Line
-	3300 2200 3400 2200
-Wire Wire Line
-	3400 2200 3700 2200
-Wire Wire Line
-	3700 2200 4200 2200
-Wire Wire Line
-	4200 2200 4800 2200
-Wire Wire Line
-	4800 2200 4900 2200
+	3000 2200 4900 2200
 Wire Wire Line
 	3300 2200 3300 2300
@@
 $EndComp
 Wire Wire Line
-	4800 4500 4800 4600
-Wire Wire Line
-	4800 4600 4800 4700
-Wire Wire Line
-	4800 4700 4800 4800
+	4800 4500 4800 4800
 Wire Wire Line
 	4800 4500 4900 4500
@@
 SCL
 Wire Wire Line
-	8500 3200 8000 3200
-Wire Wire Line
-	8000 3200 6700 3200
-Wire Wire Line
-	6700 3100 7700 3100
-Wire Wire Line
-	7700 3100 8500 3100
+	6700 3200 8500 3200
+Wire Wire Line
+	6700 3100 8500 3100
 $Comp
 L R-0603 R29
@@
 DBGRX
 Wire Wire Line
-	8500 4600 8000 4600
-Wire Wire Line
-	8000 4600 6700 4600
+	6700 4600 8500 4600
 $Comp
 L R-0603 R32

Commit message: Commit R1.0 sent to fab
Parts:
- added DS1: 5VA, smd-semi:LED-0603, symbol LED-0603
- added DS2: 5VB, smd-semi:LED-0603, symbol LED-0603
- added DS3: 3VA, smd-semi:LED-0603, symbol LED-0603
- added DS4: 3VB, smd-semi:LED-0603, symbol LED-0603
- added DS5: N12, smd-semi:LED-0603, symbol LED-0603
- added DS6: SFY, smd-semi:LED-0603, symbol LED-0603
- added R33, R34, R35: 1k, IPC7351-Nominal:RESC1608X50, symbol R-0603
Connections:
- net CLK1: now also U7.11 (OC4B/OC5B/SCK/PC5); no longer U7.12 (OC4A/OC5A/~SS~/PC4)
- net CLK2: now also U7.12 (OC4A/OC5A/~SS~/PC4); no longer U7.11 (OC4B/OC5B/SCK/PC5)
- net CLK3: now also U7.9 (OC4D/TX0/MOSI/PC7); no longer U7.10 (OC4C/RX0/MISO/PC6)
- net CLK4: now also U7.10 (OC4C/RX0/MISO/PC6); no longer U7.9 (OC4D/TX0/MOSI/PC7)
- net PG1: now also U7.25 (ADC11/TX0/PD3); no longer U7.24 (ADC12/OC5A/PD4)
- net PG2: now also U7.24 (ADC12/OC5A/PD4); no longer U7.25 (ADC11/TX0/PD3)
- net PG3: now also U7.27 (ADC9/SCL/PD1); no longer U7.26 (ADC10/RX0/PD2)
- net PG4: now also U7.26 (ADC10/RX0/PD2); no longer U7.27 (ADC9/SCL/PD1)
- net LED_A: now reaches U7.4 (ADC2/DAC0/PA2)
- net LED_A: now also R33.2
- net LED_G renamed LED_C
- net LED_C: now also R35.2
- net LED_R renamed LED_B
- net LED_B: now also R34.2
- new net: DS1.2 (A), DS3.1 (K), DS5.2 (A), DS6.1 (K), R33.1
- new net: DS1.1 (K), DS2.2 (A), DS3.2 (A), DS4.1 (K), R34.1
- new net: DS2.1 (K), DS4.2 (A), DS5.1 (K), DS6.2 (A), R35.1
Changed lines of the file:
@@
 $EndComp
 $Comp
-L GND #PWR52
+L GND #PWR51
 U 1 1 5775B96F
 P 1900 2600
-F 0 "#PWR52" H 1900 2600 30  0001 C CNN
+F 0 "#PWR51" H 1900 2600 30  0001 C CNN
 F 1 "GND" H 1900 2530 30  0001 C CNN
 F 2 "" H 1900 2600 60  0000 C CNN
@@
 $EndComp
 $Comp
-L GND #PWR53
+L GND #PWR52
 U 1 1 5775B9E7
 P 2650 2600
-F 0 "#PWR53" H 2650 2600 30  0001 C CNN
+F 0 "#PWR52" H 2650 2600 30  0001 C CNN
 F 1 "GND" H 2650 2530 30  0001 C CNN
 F 2 "" H 2650 2600 60  0000 C CNN
@@
 $EndComp
 $Comp
-L GND #PWR54
+L GND #PWR53
 U 1 1 5775BA0A
 P 3300 2600
-F 0 "#PWR54" H 3300 2600 30  0001 C CNN
+F 0 "#PWR53" H 3300 2600 30  0001 C CNN
 F 1 "GND" H 3300 2530 30  0001 C CNN
 F 2 "" H 3300 2600 60  0000 C CNN
@@
 $EndComp
 $Comp
-L +3.3 #PWR55
+L +3.3 #PWR54
 U 1 1 5775BA30
 P 3400 2150
-F 0 "#PWR55" H 3400 2200 30  0001 C CNN
+F 0 "#PWR54" H 3400 2200 30  0001 C CNN
 F 1 "+3.3" H 3400 2283 50  0000 C CNN
 F 2 "" H 3400 2150 60  0000 C CNN
@@
 Connection ~ 3700 2200
 $Comp
-L GND #PWR58
+L GND #PWR57
 U 1 1 5775BB08
 P 3700 2600
-F 0 "#PWR58" H 3700 2600 30  0001 C CNN
+F 0 "#PWR57" H 3700 2600 30  0001 C CNN
 F 1 "GND" H 3700 2530 30  0001 C CNN
 F 2 "" H 3700 2600 60  0000 C CNN
@@
 	3700 2600 3700 2500
 $Comp
-L GND #PWR59
+L GND #PWR58
 U 1 1 5775BB42
 P 4800 4800
-F 0 "#PWR59" H 4800 4800 30  0001 C CNN
+F 0 "#PWR58" H 4800 4800 30  0001 C CNN
 F 1 "GND" H 4800 4730 30  0001 C CNN
 F 2 "" H 4800 4800 60  0000 C CNN
@@
 	4900 4700 4800 4700
 Connection ~ 4800 4700
+Text HLabel 8500 3600 2    60   Output ~ 0
+CLK1
 Text HLabel 8500 3500 2    60   Output ~ 0
-CLK1
-Text HLabel 8500 3600 2    60   Output ~ 0
 CLK2
+Text HLabel 8500 3800 2    60   Output ~ 0
+CLK3
 Text HLabel 8500 3700 2    60   Output ~ 0
-CLK3
-Text HLabel 8500 3800 2    60   Output ~ 0
 CLK4
 Wire Wire Line
@@
 Connection ~ 8000 3200
 $Comp
-L +3.3 #PWR60
+L +3.3 #PWR59
 U 1 1 5775C145
 P 7700 2800
-F 0 "#PWR60" H 7700 2850 30  0001 C CNN
+F 0 "#PWR59" H 7700 2850 30  0001 C CNN
 F 1 "+3.3" H 7700 2933 50  0000 C CNN
 F 2 "" H 7700 2800 60  0000 C CNN
@@
 	7700 2800 7700 2850
 $Comp
-L +3.3 #PWR61
+L +3.3 #PWR60
 U 1 1 5775C196
 P 8000 2800
-F 0 "#PWR61" H 8000 2850 30  0001 C CNN
+F 0 "#PWR60" H 8000 2850 30  0001 C CNN
 F 1 "+3.3" H 8000 2933 50  0000 C CNN
 F 2 "" H 8000 2800 60  0000 C CNN
@@
 	2400 3800 2800 3800
 $Comp
-L +3.3 #PWR56
+L +3.3 #PWR55
 U 1 1 5775FBBE
 P 3600 3550
-F 0 "#PWR56" H 3600 3600 30  0001 C CNN
+F 0 "#PWR55" H 3600 3600 30  0001 C CNN
 F 1 "+3.3" H 3600 3683 50  0000 C CNN
 F 2 "" H 3600 3550 60  0000 C CNN
@@
 	3600 3600 3200 3600
 $Comp
-L GND #PWR57
+L GND #PWR56
 U 1 1 5775FC23
 P 3600 3850
-F 0 "#PWR57" H 3600 3850 30  0001 C CNN
+F 0 "#PWR56" H 3600 3850 30  0001 C CNN
 F 1 "GND" H 3600 3780 30  0001 C CNN
 F 2 "" H 3600 3850 60  0000 C CNN
@@
 Wire Wire Line
 	8500 4400 6700 4400
+Text HLabel 8500 4300 2    60   Input ~ 0
+PG1
 Text HLabel 8500 4400 2    60   Input ~ 0
-PG1
-Text HLabel 8500 4300 2    60   Input ~ 0
 PG2
+Text HLabel 8500 4100 2    60   Input ~ 0
+PG3
 Text HLabel 8500 4200 2    60   Input ~ 0
-PG3
-Text HLabel 8500 4100 2    60   Input ~ 0
 PG4
 Text HLabel 8500 4000 2    60   Input ~ 0
@@
 Connection ~ 8000 4600
 $Comp
-L +3.3 #PWR62
+L +3.3 #PWR61
 U 1 1 5776C60D
 P 8000 5100
-F 0 "#PWR62" H 8000 5150 30  0001 C CNN
+F 0 "#PWR61" H 8000 5150 30  0001 C CNN
 F 1 "+3.3" H 8000 5233 50  0000 C CNN
 F 2 "" H 8000 5100 60  0000 C CNN
@@
 Wire Wire Line
 	8500 3300 6700 3300
-Text HLabel 8500 2500 2    60   Output ~ 0
-LED_G
-Text HLabel 8500 2600 2    60   Output ~ 0
-LED_R
-Wire Wire Line
-	8500 2600 6700 2600
-Wire Wire Line
-	6700 2500 8500 2500
+$Comp
+L R-0603 R33
+U 1 1 5777E459
+P 5900 5700
+F 0 "R33" V 5700 5700 50  0000 C CNN
+F 1 "1k" V 5791 5700 50  0000 C CNN
+F 2 "IPC7351-Nominal:RESC1608X50" H 5900 5700 50  0001 C CNN
+F 3 "" H 5900 5750 60  0000 C CNN
+F 4 "RES SMD 1k 1% [0603]" H 6650 6250 60  0001 C CNN "BOM"
+	1    5900 5700
+	0    1    1    0
+$EndComp
+$Comp
+L R-0603 R34
+U 1 1 5777E524
+P 5900 6100
+F 0 "R34" V 5700 6100 50  0000 C CNN
+F 1 "1k" V 5791 6100 50  0000 C CNN
+F 2 "IPC7351-Nominal:RESC1608X50" H 5900 6100 50  0001 C CNN
+F 3 "" H 5900 6150 60  0000 C CNN
+F 4 "RES SMD 1k 1% [0603]" H 6650 6650 60  0001 C CNN "BOM"
+	1    5900 6100
+	0    1    1    0
+$EndComp
+$Comp
+L R-0603 R35
+U 1 1 5777E56E
+P 5900 6500
+F 0 "R35" V 5700 6500 50  0000 C CNN
+F 1 "1k" V 5791 6500 50  0000 C CNN
+F 2 "IPC7351-Nominal:RESC1608X50" H 5900 6500 50  0001 C CNN
+F 3 "" H 5900 6550 60  0000 C CNN
+F 4 "RES SMD 1k 1% [0603]" H 6650 7050 60  0001 C CNN "BOM"
+	1    5900 6500
+	0    1    1    0
+$EndComp
+$Comp
+L LED-0603 DS1
+U 1 1 5777E5A9
+P 6200 5900
+F 0 "DS1" H 6350 5946 50  0000 L CNN
+F 1 "5VA" H 6350 5855 50  0000 L CNN
+F 2 "smd-semi:LED-0603" H 6200 5750 50  0001 C CNN
+F 3 "" H 6200 5900 60  0000 C CNN
+F 4 "LED GREEN [0603]" H 6200 5650 60  0001 C CNN "BOM"
+	1    6200 5900
+	1    0    0    -1
+$EndComp
+Wire Wire Line
+	6000 5700 7600 5700
+Wire Wire Line
+	6200 5700 6200 5800
+Wire Wire Line
+	6200 6000 6200 6100
+Wire Wire Line
+	6000 6100 6800 6100
+$Comp
+L LED-0603 DS3
+U 1 1 5777E75D
+P 6700 5900
+F 0 "DS3" H 6620 5854 50  0000 R CNN
+F 1 "3VA" H 6620 5945 50  0000 R CNN
+F 2 "smd-semi:LED-0603" H 6700 5750 50  0001 C CNN
+F 3 "" H 6700 5900 60  0000 C CNN
+F 4 "LED GREEN [0603]" H 6700 5650 60  0001 C CNN "BOM"
+	1    6700 5900
+	-1   0    0    1
+$EndComp
+Wire Wire Line
+	6700 5700 6700 5800
+Connection ~ 6200 5700
+Wire Wire Line
+	6700 6100 6700 6000
+Connection ~ 6200 6100
+$Comp
+L LED-0603 DS2
+U 1 1 5777E8E6
+P 6300 6300
+F 0 "DS2" H 6450 6346 50  0000 L CNN
+F 1 "5VB" H 6450 6255 50  0000 L CNN
+F 2 "smd-semi:LED-0603" H 6300 6150 50  0001 C CNN
+F 3 "" H 6300 6300 60  0000 C CNN
+F 4 "LED GREEN [0603]" H 6300 6050 60  0001 C CNN "BOM"
+	1    6300 6300
+	1    0    0    -1
+$EndComp
+$Comp
+L LED-0603 DS4
+U 1 1 5777E934
+P 6800 6300
+F 0 "DS4" H 6720 6254 50  0000 R CNN
+F 1 "3VB" H 6720 6345 50  0000 R CNN
+F 2 "smd-semi:LED-0603" H 6800 6150 50  0001 C CNN
+F 3 "" H 6800 6300 60  0000 C CNN
+F 4 "LED GREEN [0603]" H 6800 6050 60  0001 C CNN "BOM"
+	1    6800 6300
+	-1   0    0    1
+$EndComp
+Wire Wire Line
+	6300 6200 6300 6100
+Connection ~ 6300 6100
+Wire Wire Line
+	6000 6500 7600 6500
+Wire Wire Line
+	6800 6500 6800 6400
+Wire Wire Line
+	6800 6100 6800 6200
+Connection ~ 6700 6100
+Wire Wire Line
+	6300 6400 6300 6500
+Connection ~ 6300 6500
+$Comp
+L LED-0603 DS6
+U 1 1 5777EB2F
+P 7600 6100
+F 0 "DS6" H 7520 6054 50  0000 R CNN
+F 1 "SFY" H 7520 6145 50  0000 R CNN
+F 2 "smd-semi:LED-0603" H 7600 5950 50  0001 C CNN
+F 3 "" H 7600 6100 60  0000 C CNN
+F 4 "LED RED [0603]" H 7600 5850 60  0001 C CNN "BOM"
+	1    7600 6100
+	-1   0    0    1
+$EndComp
+$Comp
+L LED-0603 DS5
+U 1 1 5777EC22
+P 7100 6100
+F 0 "DS5" H 7250 6146 50  0000 L CNN
+F 1 "N12" H 7250 6055 50  0000 L CNN
+F 2 "smd-semi:LED-0603" H 7100 5950 50  0001 C CNN
+F 3 "" H 7100 6100 60  0000 C CNN
+F 4 "LED GREEN [0603]" H 7100 5850 60  0001 C CNN "BOM"
+	1    7100 6100
+	1    0    0    -1
+$EndComp
+Wire Wire Line
+	7600 5700 7600 6000
+Connection ~ 6700 5700
+Wire Wire Line
+	7100 6000 7100 5700
+Connection ~ 7100 5700
+Wire Wire Line
+	7100 6500 7100 6200
+Connection ~ 6800 6500
+Wire Wire Line
+	7600 6500 7600 6200
+Connection ~ 7100 6500
+Text Label 5400 5700 0    60   ~ 0
+LED_A
+Wire Wire Line
+	5400 5700 5800 5700
+Text Label 5400 6100 0    60   ~ 0
+LED_B
+Wire Wire Line
+	5400 6100 5800 6100
+Text Label 5400 6500 0    60   ~ 0
+LED_C
+Wire Wire Line
+	5400 6500 5800 6500
+Text Label 7300 2600 2    60   ~ 0
+LED_B
+Wire Wire Line
+	7300 2600 6700 2600
+Text Label 7300 2500 2    60   ~ 0
+LED_C
+Text Label 7300 2400 2    60   ~ 0
+LED_A
+Wire Wire Line
+	7300 2400 6700 2400
+Wire Wire Line
+	6700 2500 7300 2500
 $EndSCHEMATC
