File: 3V3_8A.sch (KiCad schematic (older format))
At the start: 14 parts, among them Q3 CSD18503Q5A, U3 RT7258GQW

Commit message: More PCB tweaks
Parts:
- C21: value C-0603 -> 1u; BOM CAP MLCC 100pF C0G 50V 5% [0603] -> CAP MLCC 1u ≥X5R 16V 20% [0603]
- R10: value R-0603 -> 62k; BOM RES SMD 1k 5% [0603] -> RES SMD 62k 1% [0603]
- R11: value R-0603 -> 20k; BOM RES SMD 1k 5% [0603] -> RES SMD 20k 1% [0603]
- R12: value R-0603 -> 100; BOM RES SMD 1k 5% [0603] -> RES SMD 100 1% [0603]
- R9: value R-0603 -> 1k; BOM RES SMD 1k 5% [0603] -> RES SMD 1k 1% [0603]
Other:
- note added: "0.808V"
- note added: "3.32V with sense\n3.35V floating sense"
Changed lines of the file:
@@
 $Descr A4 11693 8268
 encoding utf-8
-Sheet 5 7
-Title ""
-Date ""
-Rev ""
-Comp ""
-Comment1 ""
+Sheet 4 7
+Title "3V3 8A regulator block"
+Date "2016-07-01"
+Rev "R1"
+Comp "c4757p / semianalog"
+Comment1 "C4-0 POWER SUPPLY"
 Comment2 ""
 Comment3 ""
@@
 AR Path="/57749458/57749889" Ref="L3"  Part="1"
 AR Path="/5774A2CF/57749889" Ref="L4"  Part="1"
-F 0 "L4" V 5563 3700 50  0000 C CNN
+F 0 "L3" V 5563 3700 50  0000 C CNN
 F 1 "2u2" V 5654 3700 50  0000 C CNN
 F 2 "manuf:BOURNS-SRP1238A" H 5800 3750 60  0001 C CNN
@@
 AR Path="/57749458/5774988A" Ref="C18"  Part="1"
 AR Path="/5774A2CF/5774988A" Ref="C25"  Part="1"
-F 0 "C25" H 5463 3396 50  0000 L CNN
+F 0 "C18" H 5463 3396 50  0000 L CNN
 F 1 "1u" H 5463 3305 50  0000 L CNN
 F 2 "IPC7351-Nominal:CAPC1608X55" H 5350 3350 50  0001 C CNN
@@
 AR Path="/57749458/5774988B" Ref="Q3"  Part="1"
 AR Path="/5774A2CF/5774988B" Ref="Q4"  Part="1"
-F 0 "Q4" H 5528 3996 50  0000 L CNN
+F 0 "Q3" H 5528 3996 50  0000 L CNN
 F 1 "CSD18503Q5A" H 5528 3905 50  0000 L CNN
 F 2 "manuf:TEXAS-Q5A" H 5400 3600 60  0001 C CNN
@@
 AR Path="/57749458/5774988C" Ref="#PWR26"  Part="1"
 AR Path="/5774A2CF/5774988C" Ref="#PWR34"  Part="1"
-F 0 "#PWR34" H 5450 4100 30  0001 C CNN
+F 0 "#PWR26" H 5450 4100 30  0001 C CNN
 F 1 "GND" H 5450 4030 30  0001 C CNN
 F 2 "" H 5450 4100 60  0000 C CNN
@@
 AR Path="/57749458/5774988D" Ref="U3"  Part="1"
 AR Path="/5774A2CF/5774988D" Ref="U4"  Part="1"
-F 0 "U4" H 4800 4067 50  0000 C CNN
+F 0 "U3" H 4800 4067 50  0000 C CNN
 F 1 "RT7258GQW" H 4800 3976 50  0000 C CNN
 F 2 "smd-semi:DFN50P300X400X80-15" H 4800 2500 50  0001 C CNN
@@
 AR Path="/57749458/5774988E" Ref="C17"  Part="1"
 AR Path="/5774A2CF/5774988E" Ref="C24"  Part="1"
-F 0 "C24" H 4213 4546 50  0000 L CNN
+F 0 "C17" H 4213 4546 50  0000 L CNN
 F 1 "1u" H 4213 4455 50  0000 L CNN
 F 2 "IPC7351-Nominal:CAPC1608X55" H 4100 4500 50  0001 C CNN
@@
 AR Path="/57749458/5774988F" Ref="#PWR24"  Part="1"
 AR Path="/5774A2CF/5774988F" Ref="#PWR32"  Part="1"
-F 0 "#PWR32" H 4100 4650 30  0001 C CNN
+F 0 "#PWR24" H 4100 4650 30  0001 C CNN
 F 1 "GND" H 4100 4580 30  0001 C CNN
 F 2 "" H 4100 4650 60  0000 C CNN
@@
 AR Path="/57749458/57749890" Ref="C15"  Part="1"
 AR Path="/5774A2CF/57749890" Ref="C22"  Part="1"
-F 0 "C22" H 3363 3446 50  0000 L CNN
+F 0 "C15" H 3363 3446 50  0000 L CNN
 F 1 "10u" H 3363 3355 50  0000 L CNN
 F 2 "IPC7351-Nominal:CAPC2012X70" H 3250 3400 50  0001 C CNN
@@
 AR Path="/57749458/57749891" Ref="C16"  Part="1"
 AR Path="/5774A2CF/57749891" Ref="C23"  Part="1"
-F 0 "C23" H 3763 3446 50  0000 L CNN
+F 0 "C16" H 3763 3446 50  0000 L CNN
 F 1 "10u" H 3763 3355 50  0000 L CNN
 F 2 "IPC7351-Nominal:CAPC2012X70" H 3650 3400 50  0001 C CNN
@@
 AR Path="/57749458/57749892" Ref="#PWR22"  Part="1"
 AR Path="/5774A2CF/57749892" Ref="#PWR30"  Part="1"
-F 0 "#PWR30" H 3250 3550 30  0001 C CNN
+F 0 "#PWR22" H 3250 3550 30  0001 C CNN
 F 1 "GND" H 3250 3480 30  0001 C CNN
 F 2 "" H 3250 3550 60  0000 C CNN
@@
 AR Path="/57749458/57749893" Ref="#PWR23"  Part="1"
 AR Path="/5774A2CF/57749893" Ref="#PWR31"  Part="1"
-F 0 "#PWR31" H 3650 3550 30  0001 C CNN
+F 0 "#PWR23" H 3650 3550 30  0001 C CNN
 F 1 "GND" H 3650 3480 30  0001 C CNN
 F 2 "" H 3650 3550 60  0000 C CNN
@@
 AR Path="/57749458/57749894" Ref="C19"  Part="1"
 AR Path="/5774A2CF/57749894" Ref="C26"  Part="1"
-F 0 "C26" H 6363 3946 50  0000 L CNN
+F 0 "C19" H 6363 3946 50  0000 L CNN
 F 1 "100u" H 6363 3855 50  0000 L CNN
 F 2 "IPC7351-Nominal:CAPC3225X88" H 6250 3900 50  0001 C CNN
@@
 AR Path="/57749458/57749895" Ref="#PWR27"  Part="1"
 AR Path="/5774A2CF/57749895" Ref="#PWR35"  Part="1"
-F 0 "#PWR35" H 6250 4050 30  0001 C CNN
+F 0 "#PWR27" H 6250 4050 30  0001 C CNN
 F 1 "GND" H 6250 3980 30  0001 C CNN
 F 2 "" H 6250 4050 60  0000 C CNN
@@
 AR Path="/57749458/57749896" Ref="C20"  Part="1"
 AR Path="/5774A2CF/57749896" Ref="C27"  Part="1"
-F 0 "C27" H 6813 3946 50  0000 L CNN
+F 0 "C20" H 6813 3946 50  0000 L CNN
 F 1 "100u" H 6813 3855 50  0000 L CNN
 F 2 "IPC7351-Nominal:CAPC3225X88" H 6700 3900 50  0001 C CNN
@@
 AR Path="/57749458/57749897" Ref="#PWR28"  Part="1"
 AR Path="/5774A2CF/57749897" Ref="#PWR36"  Part="1"
-F 0 "#PWR36" H 6700 4050 30  0001 C CNN
+F 0 "#PWR28" H 6700 4050 30  0001 C CNN
 F 1 "GND" H 6700 3980 30  0001 C CNN
 F 2 "" H 6700 4050 60  0000 C CNN
@@
 AR Path="/57749458/57749898" Ref="R9"  Part="1"
 AR Path="/5774A2CF/57749898" Ref="R13"  Part="1"
-F 0 "R13" H 7163 3946 50  0000 L CNN
-F 1 "R-0603" H 7163 3855 50  0000 L CNN
+F 0 "R9" H 7163 3946 50  0000 L CNN
+F 1 "1k" H 7163 3855 50  0000 L CNN
 F 2 "IPC7351-Nominal:RESC1608X50" H 7100 3900 50  0001 C CNN
 F 3 "" H 7100 3950 60  0000 C CNN
-F 4 "RES SMD 1k 5% [0603]" H 7850 4450 60  0001 C CNN "BOM"
+F 4 "RES SMD 1k 1% [0603]" H 7850 4450 60  0001 C CNN "BOM"
 	1    7100 3900
 	1    0    0    -1
@@
 AR Path="/57749458/57749899" Ref="R10"  Part="1"
 AR Path="/5774A2CF/57749899" Ref="R14"  Part="1"
-F 0 "R14" H 7163 4346 50  0000 L CNN
-F 1 "R-0603" H 7163 4255 50  0000 L CNN
+F 0 "R10" H 7163 4346 50  0000 L CNN
+F 1 "62k" H 7163 4255 50  0000 L CNN
 F 2 "IPC7351-Nominal:RESC1608X50" H 7100 4300 50  0001 C CNN
 F 3 "" H 7100 4350 60  0000 C CNN
-F 4 "RES SMD 1k 5% [0603]" H 7850 4850 60  0001 C CNN "BOM"
+F 4 "RES SMD 62k 1% [0603]" H 7850 4850 60  0001 C CNN "BOM"
 	1    7100 4300
 	1    0    0    -1
@@
 AR Path="/57749458/5774989A" Ref="R11"  Part="1"
 AR Path="/5774A2CF/5774989A" Ref="R15"  Part="1"
-F 0 "R15" H 7163 4746 50  0000 L CNN
-F 1 "R-0603" H 7163 4655 50  0000 L CNN
+F 0 "R11" H 7163 4746 50  0000 L CNN
+F 1 "20k" H 7163 4655 50  0000 L CNN
 F 2 "IPC7351-Nominal:RESC1608X50" H 7100 4700 50  0001 C CNN
 F 3 "" H 7100 4750 60  0000 C CNN
-F 4 "RES SMD 1k 5% [0603]" H 7850 5250 60  0001 C CNN "BOM"
+F 4 "RES SMD 20k 1% [0603]" H 7850 5250 60  0001 C CNN "BOM"
 	1    7100 4700
 	1    0    0    -1
@@
 AR Path="/57749458/5774989B" Ref="C21"  Part="1"
 AR Path="/5774A2CF/5774989B" Ref="C28"  Part="1"
-F 0 "C28" H 7713 3946 50  0000 L CNN
-F 1 "C-0603" H 7713 3855 50  0000 L CNN
+F 0 "C21" H 7713 3946 50  0000 L CNN
+F 1 "1u" H 7713 3855 50  0000 L CNN
 F 2 "IPC7351-Nominal:CAPC1608X55" H 7600 3900 50  0001 C CNN
 F 3 "" H 7590 3875 60  0000 C CNN
-F 4 "CAP MLCC 100pF C0G 50V 5% [0603]" H 8400 4450 60  0001 C CNN "BOM"
+F 4 "CAP MLCC 1u ≥X5R 16V 20% [0603]" H 8400 4450 60  0001 C CNN "BOM"
 	1    7600 3900
 	1    0    0    -1
@@
 AR Path="/57749458/5774989C" Ref="R12"  Part="1"
 AR Path="/5774A2CF/5774989C" Ref="R16"  Part="1"
-F 0 "R16" V 8050 4100 50  0000 C CNN
-F 1 "R-0603" V 8141 4100 50  0000 C CNN
+F 0 "R12" V 8050 4100 50  0000 C CNN
+F 1 "100" V 8141 4100 50  0000 C CNN
 F 2 "IPC7351-Nominal:RESC1608X50" H 8250 4100 50  0001 C CNN
 F 3 "" H 8250 4150 60  0000 C CNN
-F 4 "RES SMD 1k 5% [0603]" H 9000 4650 60  0001 C CNN "BOM"
+F 4 "RES SMD 100 1% [0603]" H 9000 4650 60  0001 C CNN "BOM"
 	1    8250 4100
 	0    1    1    0
@@
 AR Path="/57749458/5774989D" Ref="#PWR29"  Part="1"
 AR Path="/5774A2CF/5774989D" Ref="#PWR37"  Part="1"
-F 0 "#PWR37" H 7100 4850 30  0001 C CNN
+F 0 "#PWR29" H 7100 4850 30  0001 C CNN
 F 1 "GND" H 7100 4780 30  0001 C CNN
 F 2 "" H 7100 4850 60  0000 C CNN
@@
 AR Path="/57749458/5774989E" Ref="#PWR25"  Part="1"
 AR Path="/5774A2CF/5774989E" Ref="#PWR33"  Part="1"
-F 0 "#PWR33" H 4350 4350 30  0001 C CNN
+F 0 "#PWR25" H 4350 4350 30  0001 C CNN
 F 1 "GND" H 4350 4280 30  0001 C CNN
 F 2 "" H 4350 4350 60  0000 C CNN
@@
 IN
 Connection ~ 3250 3200
+Text Notes 7800 3500 0    60   ~ 0
+3.32V with sense\n3.35V floating sense
+Text Notes 6550 4400 0    60   ~ 0
+0.808V
 $EndSCHEMATC

Commit message: Final rev take 2
Changed lines of the file:
@@
 AR Path="/57749458/57749889" Ref="L3"  Part="1"
 AR Path="/5774A2CF/57749889" Ref="L4"  Part="1"
-F 0 "L3" V 5563 3700 50  0000 C CNN
+F 0 "L4" V 5563 3700 50  0000 C CNN
 F 1 "2u2" V 5654 3700 50  0000 C CNN
 F 2 "manuf:BOURNS-SRP1238A" H 5800 3750 60  0001 C CNN
@@
 AR Path="/57749458/5774988A" Ref="C18"  Part="1"
 AR Path="/5774A2CF/5774988A" Ref="C25"  Part="1"
-F 0 "C18" H 5463 3396 50  0000 L CNN
+F 0 "C25" H 5463 3396 50  0000 L CNN
 F 1 "1u" H 5463 3305 50  0000 L CNN
 F 2 "IPC7351-Nominal:CAPC1608X55" H 5350 3350 50  0001 C CNN
@@
 AR Path="/57749458/5774988B" Ref="Q3"  Part="1"
 AR Path="/5774A2CF/5774988B" Ref="Q4"  Part="1"
-F 0 "Q3" H 5528 3996 50  0000 L CNN
+F 0 "Q4" H 5528 3996 50  0000 L CNN
 F 1 "CSD18503Q5A" H 5528 3905 50  0000 L CNN
 F 2 "manuf:TEXAS-Q5A" H 5400 3600 60  0001 C CNN
@@
 AR Path="/57749458/5774988C" Ref="#PWR25"  Part="1"
 AR Path="/5774A2CF/5774988C" Ref="#PWR33"  Part="1"
-F 0 "#PWR25" H 5450 4100 30  0001 C CNN
+F 0 "#PWR33" H 5450 4100 30  0001 C CNN
 F 1 "GND" H 5450 4030 30  0001 C CNN
 F 2 "" H 5450 4100 60  0000 C CNN
@@
 AR Path="/57749458/5774988D" Ref="U3"  Part="1"
 AR Path="/5774A2CF/5774988D" Ref="U4"  Part="1"
-F 0 "U3" H 4800 4067 50  0000 C CNN
+F 0 "U4" H 4800 4067 50  0000 C CNN
 F 1 "RT7258GQW" H 4800 3976 50  0000 C CNN
 F 2 "smd-semi:DFN50P300X400X80-15" H 4800 2500 50  0001 C CNN
@@
 AR Path="/57749458/5774988E" Ref="C17"  Part="1"
 AR Path="/5774A2CF/5774988E" Ref="C24"  Part="1"
-F 0 "C17" H 4213 4546 50  0000 L CNN
+F 0 "C24" H 4213 4546 50  0000 L CNN
 F 1 "1u" H 4213 4455 50  0000 L CNN
 F 2 "IPC7351-Nominal:CAPC1608X55" H 4100 4500 50  0001 C CNN
@@
 AR Path="/57749458/5774988F" Ref="#PWR23"  Part="1"
 AR Path="/5774A2CF/5774988F" Ref="#PWR31"  Part="1"
-F 0 "#PWR23" H 4100 4650 30  0001 C CNN
+F 0 "#PWR31" H 4100 4650 30  0001 C CNN
 F 1 "GND" H 4100 4580 30  0001 C CNN
 F 2 "" H 4100 4650 60  0000 C CNN
@@
 AR Path="/57749458/57749890" Ref="C15"  Part="1"
 AR Path="/5774A2CF/57749890" Ref="C22"  Part="1"
-F 0 "C15" H 3363 3446 50  0000 L CNN
+F 0 "C22" H 3363 3446 50  0000 L CNN
 F 1 "10u" H 3363 3355 50  0000 L CNN
 F 2 "IPC7351-Nominal:CAPC2012X70" H 3250 3400 50  0001 C CNN
@@
 AR Path="/57749458/57749891" Ref="C16"  Part="1"
 AR Path="/5774A2CF/57749891" Ref="C23"  Part="1"
-F 0 "C16" H 3763 3446 50  0000 L CNN
+F 0 "C23" H 3763 3446 50  0000 L CNN
 F 1 "10u" H 3763 3355 50  0000 L CNN
 F 2 "IPC7351-Nominal:CAPC2012X70" H 3650 3400 50  0001 C CNN
@@
 AR Path="/57749458/57749892" Ref="#PWR21"  Part="1"
 AR Path="/5774A2CF/57749892" Ref="#PWR29"  Part="1"
-F 0 "#PWR21" H 3250 3550 30  0001 C CNN
+F 0 "#PWR29" H 3250 3550 30  0001 C CNN
 F 1 "GND" H 3250 3480 30  0001 C CNN
 F 2 "" H 3250 3550 60  0000 C CNN
@@
 AR Path="/57749458/57749893" Ref="#PWR22"  Part="1"
 AR Path="/5774A2CF/57749893" Ref="#PWR30"  Part="1"
-F 0 "#PWR22" H 3650 3550 30  0001 C CNN
+F 0 "#PWR30" H 3650 3550 30  0001 C CNN
 F 1 "GND" H 3650 3480 30  0001 C CNN
 F 2 "" H 3650 3550 60  0000 C CNN
@@
 AR Path="/57749458/57749894" Ref="C19"  Part="1"
 AR Path="/5774A2CF/57749894" Ref="C26"  Part="1"
-F 0 "C19" H 6363 3946 50  0000 L CNN
+F 0 "C26" H 6363 3946 50  0000 L CNN
 F 1 "100u" H 6363 3855 50  0000 L CNN
 F 2 "IPC7351-Nominal:CAPC3225X88" H 6250 3900 50  0001 C CNN
@@
 AR Path="/57749458/57749895" Ref="#PWR26"  Part="1"
 AR Path="/5774A2CF/57749895" Ref="#PWR34"  Part="1"
-F 0 "#PWR26" H 6250 4050 30  0001 C CNN
+F 0 "#PWR34" H 6250 4050 30  0001 C CNN
 F 1 "GND" H 6250 3980 30  0001 C CNN
 F 2 "" H 6250 4050 60  0000 C CNN
@@
 AR Path="/57749458/57749896" Ref="C20"  Part="1"
 AR Path="/5774A2CF/57749896" Ref="C27"  Part="1"
-F 0 "C20" H 6813 3946 50  0000 L CNN
+F 0 "C27" H 6813 3946 50  0000 L CNN
 F 1 "100u" H 6813 3855 50  0000 L CNN
 F 2 "IPC7351-Nominal:CAPC3225X88" H 6700 3900 50  0001 C CNN
@@
 AR Path="/57749458/57749897" Ref="#PWR27"  Part="1"
 AR Path="/5774A2CF/57749897" Ref="#PWR35"  Part="1"
-F 0 "#PWR27" H 6700 4050 30  0001 C CNN
+F 0 "#PWR35" H 6700 4050 30  0001 C CNN
 F 1 "GND" H 6700 3980 30  0001 C CNN
 F 2 "" H 6700 4050 60  0000 C CNN
@@
 AR Path="/57749458/57749898" Ref="R9"  Part="1"
 AR Path="/5774A2CF/57749898" Ref="R13"  Part="1"
-F 0 "R9" H 7163 3946 50  0000 L CNN
+F 0 "R13" H 7163 3946 50  0000 L CNN
 F 1 "1k" H 7163 3855 50  0000 L CNN
 F 2 "IPC7351-Nominal:RESC1608X50" H 7100 3900 50  0001 C CNN
@@
 AR Path="/57749458/57749899" Ref="R10"  Part="1"
 AR Path="/5774A2CF/57749899" Ref="R14"  Part="1"
-F 0 "R10" H 7163 4346 50  0000 L CNN
+F 0 "R14" H 7163 4346 50  0000 L CNN
 F 1 "62k" H 7163 4255 50  0000 L CNN
 F 2 "IPC7351-Nominal:RESC1608X50" H 7100 4300 50  0001 C CNN
@@
 AR Path="/57749458/5774989A" Ref="R11"  Part="1"
 AR Path="/5774A2CF/5774989A" Ref="R15"  Part="1"
-F 0 "R11" H 7163 4746 50  0000 L CNN
+F 0 "R15" H 7163 4746 50  0000 L CNN
 F 1 "20k" H 7163 4655 50  0000 L CNN
 F 2 "IPC7351-Nominal:RESC1608X50" H 7100 4700 50  0001 C CNN
@@
 AR Path="/57749458/5774989B" Ref="C21"  Part="1"
 AR Path="/5774A2CF/5774989B" Ref="C28"  Part="1"
-F 0 "C21" H 7713 3946 50  0000 L CNN
+F 0 "C28" H 7713 3946 50  0000 L CNN
 F 1 "1u" H 7713 3855 50  0000 L CNN
 F 2 "IPC7351-Nominal:CAPC1608X55" H 7600 3900 50  0001 C CNN
@@
 AR Path="/57749458/5774989C" Ref="R12"  Part="1"
 AR Path="/5774A2CF/5774989C" Ref="R16"  Part="1"
-F 0 "R12" V 8050 4100 50  0000 C CNN
+F 0 "R16" V 8050 4100 50  0000 C CNN
 F 1 "100" V 8141 4100 50  0000 C CNN
 F 2 "IPC7351-Nominal:RESC1608X50" H 8250 4100 50  0001 C CNN
@@
 AR Path="/57749458/5774989D" Ref="#PWR28"  Part="1"
 AR Path="/5774A2CF/5774989D" Ref="#PWR36"  Part="1"
-F 0 "#PWR28" H 7100 4850 30  0001 C CNN
+F 0 "#PWR36" H 7100 4850 30  0001 C CNN
 F 1 "GND" H 7100 4780 30  0001 C CNN
 F 2 "" H 7100 4850 60  0000 C CNN
@@
 AR Path="/57749458/5774989E" Ref="#PWR24"  Part="1"
 AR Path="/5774A2CF/5774989E" Ref="#PWR32"  Part="1"
-F 0 "#PWR24" H 4350 4350 30  0001 C CNN
+F 0 "#PWR32" H 4350 4350 30  0001 C CNN
 F 1 "GND" H 4350 4280 30  0001 C CNN
 F 2 "" H 4350 4350 60  0000 C CNN
