File: N12V_1A.sch (KiCad schematic (older format))
At the start: 33 parts, among them Q5 BSS84, Q6 2N7002, Q7 2N7002, U5 74HCT1G02, U6 RT7258GQW

Commit message: Commit R1.0 sent to fab
Parts:
- C38: value C-0603 -> DNP
- R25, R28: value R-0603 -> 0R
- R26: value R-0603 -> 3k6; BOM RES SMD 1k 5% [0603] -> RES SMD 3k6 1% [0603]
- R27: value R-0603 -> 51k; BOM RES SMD 1k 5% [0603] -> RES SMD 51k 1% [0603]
Changed lines of the file:
@@
 $EndComp
 $Comp
-L GND #PWR45
+L GND #PWR44
 U 1 1 5774C2EE
 P 5800 3600
-F 0 "#PWR45" H 5800 3600 30  0001 C CNN
+F 0 "#PWR44" H 5800 3600 30  0001 C CNN
 F 1 "GND" H 5800 3530 30  0001 C CNN
 F 2 "" H 5800 3600 60  0000 C CNN
@@
 $EndComp
 $Comp
-L GND #PWR46
+L GND #PWR45
 U 1 1 5774C4A7
 P 6600 3600
-F 0 "#PWR46" H 6600 3600 30  0001 C CNN
+F 0 "#PWR45" H 6600 3600 30  0001 C CNN
 F 1 "GND" H 6600 3530 30  0001 C CNN
 F 2 "" H 6600 3600 60  0000 C CNN
@@
 $EndComp
 $Comp
-L GND #PWR47
+L GND #PWR46
 U 1 1 5774C4F2
 P 7000 3600
-F 0 "#PWR47" H 7000 3600 30  0001 C CNN
+F 0 "#PWR46" H 7000 3600 30  0001 C CNN
 F 1 "GND" H 7000 3530 30  0001 C CNN
 F 2 "" H 7000 3600 60  0000 C CNN
@@
 $EndComp
 $Comp
-L GND #PWR48
+L GND #PWR47
 U 1 1 5774C536
 P 7400 3600
-F 0 "#PWR48" H 7400 3600 30  0001 C CNN
+F 0 "#PWR47" H 7400 3600 30  0001 C CNN
 F 1 "GND" H 7400 3530 30  0001 C CNN
 F 2 "" H 7400 3600 60  0000 C CNN
@@
 $EndComp
 $Comp
-L GND #PWR49
+L GND #PWR48
 U 1 1 5774C57B
 P 7800 3600
-F 0 "#PWR49" H 7800 3600 30  0001 C CNN
+F 0 "#PWR48" H 7800 3600 30  0001 C CNN
 F 1 "GND" H 7800 3530 30  0001 C CNN
 F 2 "" H 7800 3600 60  0000 C CNN
@@
 $EndComp
 $Comp
-L GND #PWR51
+L GND #PWR50
 U 1 1 5774C715
 P 9900 3600
-F 0 "#PWR51" H 9900 3600 30  0001 C CNN
+F 0 "#PWR50" H 9900 3600 30  0001 C CNN
 F 1 "GND" H 9900 3530 30  0001 C CNN
 F 2 "" H 9900 3600 60  0000 C CNN
@@
 P 8400 3600
 F 0 "R25" H 8463 3646 50  0000 L CNN
-F 1 "R-0603" H 8463 3555 50  0000 L CNN
+F 1 "0R" H 8463 3555 50  0000 L CNN
 F 2 "IPC7351-Nominal:RESC1608X50" H 8400 3600 50  0001 C CNN
 F 3 "" H 8400 3650 60  0000 C CNN
@@
 P 9500 3800
 F 0 "R28" V 9300 3800 50  0000 C CNN
-F 1 "R-0603" V 9391 3800 50  0000 C CNN
+F 1 "0R" V 9391 3800 50  0000 C CNN
 F 2 "IPC7351-Nominal:RESC1608X50" H 9500 3800 50  0001 C CNN
 F 3 "" H 9500 3850 60  0000 C CNN
@@
 P 8400 4000
 F 0 "R26" H 8337 3954 50  0000 R CNN
-F 1 "R-0603" H 8337 4045 50  0000 R CNN
+F 1 "3k6" H 8337 4045 50  0000 R CNN
 F 2 "IPC7351-Nominal:RESC1608X50" H 8400 4000 50  0001 C CNN
 F 3 "" H 8400 4050 60  0000 C CNN
-F 4 "RES SMD 1k 5% [0603]" H 9150 4550 60  0001 C CNN "BOM"
+F 4 "RES SMD 3k6 1% [0603]" H 9150 4550 60  0001 C CNN "BOM"
 	1    8400 4000
 	-1   0    0    1
@@
 P 8400 4400
 F 0 "R27" H 8337 4354 50  0000 R CNN
-F 1 "R-0603" H 8337 4445 50  0000 R CNN
+F 1 "51k" H 8337 4445 50  0000 R CNN
 F 2 "IPC7351-Nominal:RESC1608X50" H 8400 4400 50  0001 C CNN
 F 3 "" H 8400 4450 60  0000 C CNN
-F 4 "RES SMD 1k 5% [0603]" H 9150 4950 60  0001 C CNN "BOM"
+F 4 "RES SMD 51k 1% [0603]" H 9150 4950 60  0001 C CNN "BOM"
 	1    8400 4400
 	-1   0    0    1
 $EndComp
 $Comp
-L GND #PWR50
+L GND #PWR49
 U 1 1 5774CC45
 P 8400 4600
-F 0 "#PWR50" H 8400 4600 30  0001 C CNN
+F 0 "#PWR49" H 8400 4600 30  0001 C CNN
 F 1 "GND" H 8400 4530 30  0001 C CNN
 F 2 "" H 8400 4600 60  0000 C CNN
@@
 $EndComp
 $Comp
-L GND #PWR43
+L GND #PWR42
 U 1 1 5774CFE4
 P 4000 3050
-F 0 "#PWR43" H 4000 3050 30  0001 C CNN
+F 0 "#PWR42" H 4000 3050 30  0001 C CNN
 F 1 "GND" H 4000 2980 30  0001 C CNN
 F 2 "" H 4000 3050 60  0000 C CNN
@@
 $EndComp
 $Comp
-L GND #PWR42
+L GND #PWR41
 U 1 1 5774DF18
 P 2750 4200
-F 0 "#PWR42" H 2750 4200 30  0001 C CNN
+F 0 "#PWR41" H 2750 4200 30  0001 C CNN
 F 1 "GND" H 2750 4130 30  0001 C CNN
 F 2 "" H 2750 4200 60  0000 C CNN
@@
 $EndComp
 $Comp
-L GND #PWR38
+L GND #PWR37
 U 1 1 5774E3F4
 P 1600 5150
-F 0 "#PWR38" H 1600 5150 30  0001 C CNN
+F 0 "#PWR37" H 1600 5150 30  0001 C CNN
 F 1 "GND" H 1600 5080 30  0001 C CNN
 F 2 "" H 1600 5150 60  0000 C CNN
@@
 $EndComp
 $Comp
-L GND #PWR41
+L GND #PWR40
 U 1 1 5774EF0B
 P 2700 3200
-F 0 "#PWR41" H 2700 3200 30  0001 C CNN
+F 0 "#PWR40" H 2700 3200 30  0001 C CNN
 F 1 "GND" H 2700 3130 30  0001 C CNN
 F 2 "" H 2700 3200 60  0000 C CNN
@@
 $EndComp
 $Comp
-L +3.3 #PWR39
+L +3.3 #PWR38
 U 1 1 5774F3B7
 P 2400 5150
-F 0 "#PWR39" H 2400 5200 30  0001 C CNN
+F 0 "#PWR38" H 2400 5200 30  0001 C CNN
 F 1 "+3.3" H 2400 5283 50  0000 C CNN
 F 2 "" H 2400 5150 60  0000 C CNN
@@
 $EndComp
 $Comp
-L GND #PWR40
+L GND #PWR39
 U 1 1 5774F534
 P 2400 6250
-F 0 "#PWR40" H 2400 6250 30  0001 C CNN
+F 0 "#PWR39" H 2400 6250 30  0001 C CNN
 F 1 "GND" H 2400 6180 30  0001 C CNN
 F 2 "" H 2400 6250 60  0000 C CNN
@@
 Wire Wire Line
 	3800 3500 4700 3500
-Wire Wire Line
-	3800 3500 3800 3250
 Wire Wire Line
 	4000 3250 4000 3200
@@
 P 8900 3600
 F 0 "C38" H 9013 3646 50  0000 L CNN
-F 1 "C-0603" H 9013 3555 50  0000 L CNN
+F 1 "DNP" H 9013 3555 50  0000 L CNN
 F 2 "IPC7351-Nominal:CAPC1608X55" H 8900 3600 50  0001 C CNN
 F 3 "" H 8890 3575 60  0000 C CNN
@@
 Connection ~ 4350 2700
 $Comp
-L GND #PWR44
+L GND #PWR43
 U 1 1 5775318F
 P 4350 3050
-F 0 "#PWR44" H 4350 3050 30  0001 C CNN
+F 0 "#PWR43" H 4350 3050 30  0001 C CNN
 F 1 "GND" H 4350 2980 30  0001 C CNN
 F 2 "" H 4350 3050 60  0000 C CNN
@@
 Wire Wire Line
 	4350 3050 4350 3000
+Wire Wire Line
+	3800 3500 3800 3250
 $EndSCHEMATC

Commit message: Final rev take 2
Parts:
- added D3: MBRD1035CTLT4G, symbol SCHOTTKY-CK
- added R36: 5k1, IPC7351-Nominal:RESC1608X50, symbol R-0603
- added R37: 100k, IPC7351-Nominal:RESC1608X50, symbol R-0603
- R17: value R-0805 -> R03; BOM RES SMD 1k 5% [0805] -> RES SMD R03 1% [0805]
- R18: value R-0805 -> R03; BOM RES SMD 1k 5% [0805] -> RES SMD R03 5% [0805]
- U5: value 74HCT1G02 -> 74HC1G02; BOM DIST DIGIKEY 568-8172-1-ND -> DIST DIGIKEY MC74HC1G02DFT2GOSCT-ND
Connections:
- net at Q7.2, R24.1: now also R36.1; no longer U6.2 (PG)
- new net: R36.2, U6.2 (PG)
Other:
- note added: "REV2: add this diode here"
- note added: "REV2: add this res here"
- moved on the sheet: R17, R18
Changed lines of the file:
@@
 L R-0805 R18
 U 1 1 5774D064
-P 1600 2700
-F 0 "R18" V 1400 2700 50  0000 C CNN
-F 1 "R-0805" V 1491 2700 50  0000 C CNN
-F 2 "IPC7351-Nominal:RESC2012X50" H 1600 2700 50  0001 C CNN
-F 3 "" H 1600 2750 60  0000 C CNN
-F 4 "RES SMD 1k 5% [0805]" H 2350 3250 60  0001 C CNN "BOM"
-	1    1600 2700
+P 1900 2700
+F 0 "R18" V 1700 2700 50  0000 C CNN
+F 1 "R03" V 1791 2700 50  0000 C CNN
+F 2 "IPC7351-Nominal:RESC2012X50" H 1900 2700 50  0001 C CNN
+F 3 "" H 1900 2750 60  0000 C CNN
+F 4 "RES SMD R03 5% [0805]" H 2650 3250 60  0001 C CNN "BOM"
+	1    1900 2700
 	0    1    1    0
 $EndComp
@@
 L R-0805 R17
 U 1 1 5774D12E
-P 1600 2400
-F 0 "R17" V 1400 2400 50  0000 C CNN
-F 1 "R-0805" V 1491 2400 50  0000 C CNN
-F 2 "IPC7351-Nominal:RESC2012X50" H 1600 2400 50  0001 C CNN
-F 3 "" H 1600 2450 60  0000 C CNN
-F 4 "RES SMD 1k 5% [0805]" H 2350 2950 60  0001 C CNN "BOM"
-	1    1600 2400
+P 1900 2400
+F 0 "R17" V 1700 2400 50  0000 C CNN
+F 1 "R03" V 1791 2400 50  0000 C CNN
+F 2 "IPC7351-Nominal:RESC2012X50" H 1900 2400 50  0001 C CNN
+F 3 "" H 1900 2450 60  0000 C CNN
+F 4 "RES SMD R03 1% [0805]" H 2650 2950 60  0001 C CNN "BOM"
+	1    1900 2400
 	0    1    1    0
 $EndComp
@@
 P 2450 3600
 F 0 "U5" H 2400 3333 50  0000 C CNN
-F 1 "74HCT1G02" H 2400 3424 50  0000 C CNN
+F 1 "74HC1G02" H 2400 3424 50  0000 C CNN
 F 2 "smd-semi:SC-70-5" H 2450 3450 50  0001 C CNN
 F 3 "" H 2250 3600 60  0000 C CNN
-F 4 "DIST DIGIKEY 568-8172-1-ND" H 2450 3600 60  0001 C CNN "BOM"
+F 4 "DIST DIGIKEY MC74HC1G02DFT2GOSCT-ND" H 2450 3600 60  0001 C CNN "BOM"
 	1    2450 3600
 	1    0    0    1
@@
 U 1 1 5774E96B
 P 3850 3150
-F 0 "Q7" H 3977 3196 50  0000 L CNN
-F 1 "2N7002" H 3977 3105 50  0000 L CNN
+F 0 "Q7" H 4000 3300 50  0000 L CNN
+F 1 "2N7002" H 4000 3200 50  0000 L CNN
 F 2 "smd-semi:SOT-23" H 3850 3000 50  0001 C CNN
 F 3 "" H 3850 3150 60  0000 C CNN
@@
 P 2400 5300
 F 0 "U5" H 2530 4946 50  0000 L CNN
-F 1 "74HCT1G02" H 2530 4855 50  0000 L CNN
+F 1 "74HC1G02" H 2530 4855 50  0000 L CNN
 F 2 "smd-semi:SC-70-5" H 2400 5150 50  0001 C CNN
 F 3 "" H 2200 5300 60  0000 C CNN
-F 4 "DIST DIGIKEY 568-8172-1-ND" H 2400 5300 60  0001 C CNN "BOM"
+F 4 "DIST DIGIKEY MC74HC1G02DFT2GOSCT-ND" H 2400 5300 60  0001 C CNN "BOM"
 	2    2400 5300
 	1    0    0    -1
@@
 $EndComp
 Wire Wire Line
-	5500 3200 6100 3200
+	5500 3200 5600 3200
+Wire Wire Line
+	5600 3200 5700 3200
+Wire Wire Line
+	5700 3200 5800 3200
+Wire Wire Line
+	5800 3200 6100 3200
 Wire Wire Line
 	5800 3200 5800 3300
 Wire Wire Line
-	5600 3000 5600 3200
+	5600 3000 5600 3100
+Wire Wire Line
+	5600 3100 5600 3200
 Wire Wire Line
 	5600 3000 5500 3000
@@
 	5800 3600 5800 3500
 Wire Wire Line
-	6300 3200 9500 3200
+	6300 3200 6600 3200
+Wire Wire Line
+	6600 3200 7000 3200
+Wire Wire Line
+	7000 3200 7400 3200
+Wire Wire Line
+	7400 3200 7800 3200
+Wire Wire Line
+	7800 3200 8200 3200
+Wire Wire Line
+	8200 3200 8400 3200
+Wire Wire Line
+	8400 3200 8900 3200
+Wire Wire Line
+	8900 3200 9500 3200
 Wire Wire Line
 	7800 3200 7800 3300
@@
 Connection ~ 7800 3200
 Wire Wire Line
-	9700 3200 10300 3200
+	9700 3200 9900 3200
+Wire Wire Line
+	9900 3200 10300 3200
 Wire Wire Line
 	9900 3200 9900 3300
@@
 	8900 3700 8900 3800
 Wire Wire Line
-	8400 3800 9400 3800
-Wire Wire Line
-	8400 3700 8400 3900
+	8400 3800 8900 3800
+Wire Wire Line
+	8900 3800 9400 3800
+Wire Wire Line
+	8400 3700 8400 3800
+Wire Wire Line
+	8400 3800 8400 3900
 Connection ~ 8900 3800
 Connection ~ 8400 3800
 Wire Wire Line
-	8400 4100 8400 4300
+	8400 4100 8400 4200
+Wire Wire Line
+	8400 4200 8400 4300
 Wire Wire Line
 	8400 4500 8400 4600
@@
 	8200 4500 8200 3200
 Wire Wire Line
-	3100 4500 8200 4500
-Wire Wire Line
-	4600 3700 4600 4500
+	3100 4500 3400 4500
+Wire Wire Line
+	3400 4500 4300 4500
+Wire Wire Line
+	4300 4500 4600 4500
+Wire Wire Line
+	4600 4500 8200 4500
+Wire Wire Line
+	4600 3700 4600 3800
+Wire Wire Line
+	4600 3800 4600 4500
 Wire Wire Line
 	4600 3700 4700 3700
@@
 Connection ~ 4600 3800
 Wire Wire Line
-	1700 2700 4700 2700
+	2000 2700 2200 2700
+Wire Wire Line
+	2200 2700 2300 2700
+Wire Wire Line
+	2300 2700 4000 2700
+Wire Wire Line
+	4000 2700 4350 2700
+Wire Wire Line
+	4350 2700 4600 2700
+Wire Wire Line
+	4600 2700 4700 2700
 Wire Wire Line
 	4000 2700 4000 2800
 Wire Wire Line
-	4600 2700 4600 2900
+	4600 2700 4600 2800
+Wire Wire Line
+	4600 2800 4600 2900
 Wire Wire Line
 	4600 2900 4700 2900
@@
 Connection ~ 4000 2700
 Wire Wire Line
-	1700 2400 1900 2400
-Wire Wire Line
-	1900 2400 1900 2700
-Connection ~ 1900 2700
-Wire Wire Line
-	3900 3200 4700 3200
+	2000 2400 2200 2400
+Wire Wire Line
+	2200 2400 2200 2700
+Connection ~ 2200 2700
+Wire Wire Line
+	3900 3200 4000 3200
+Wire Wire Line
+	4000 3200 4300 3200
+Wire Wire Line
+	4300 3200 4700 3200
 Wire Wire Line
 	4300 3200 4300 3800
@@
 	3100 3600 3000 3600
 Wire Wire Line
-	3300 3600 4700 3600
+	3300 3600 3400 3600
+Wire Wire Line
+	3400 3600 4700 3600
 Wire Wire Line
 	3400 3900 3400 3600
 Connection ~ 3400 3600
 Wire Wire Line
-	2900 4050 3300 4050
+	2900 4050 3100 4050
+Wire Wire Line
+	3100 4050 3300 4050
 Wire Wire Line
 	3100 4050 3100 4200
@@
 	2700 4050 1900 4050
 Wire Wire Line
-	1900 3550 1900 4500
-Wire Wire Line
-	1400 3550 2100 3550
+	1900 3550 1900 4050
+Wire Wire Line
+	1900 4050 1900 4500
+Wire Wire Line
+	1400 3550 1900 3550
+Wire Wire Line
+	1900 3550 2100 3550
 Wire Wire Line
 	2750 4200 2750 4150
@@
 	1600 4900 1600 4800
 Wire Wire Line
-	1600 4400 1600 4600
+	1600 4400 1600 4500
+Wire Wire Line
+	1600 4500 1600 4600
 Wire Wire Line
 	1900 4500 1600 4500
@@
 	1600 4200 1600 3100
 Wire Wire Line
-	1600 3100 2000 3100
-Wire Wire Line
-	2000 3100 2000 2700
-Connection ~ 2000 2700
+	1600 3100 2300 3100
+Wire Wire Line
+	2300 3100 2300 2700
+Connection ~ 2300 2700
 Connection ~ 4300 3200
-Wire Wire Line
-	3800 3500 4700 3500
 Wire Wire Line
 	4000 3250 4000 3200
@@
 	3800 2900 3800 3050
 Wire Wire Line
-	2600 2900 3800 2900
+	2600 2900 3200 2900
+Wire Wire Line
+	3200 2900 3800 2900
 Wire Wire Line
 	3000 3200 3200 3200
@@
 	2700 3200 2800 3200
 Wire Wire Line
-	2400 5150 2400 5300
+	2400 5150 2400 5200
+Wire Wire Line
+	2400 5200 2400 5300
 Wire Wire Line
 	2400 5200 3100 5200
@@
 Connection ~ 2400 5200
 Wire Wire Line
-	2400 6100 2400 6250
+	2400 6100 2400 6200
+Wire Wire Line
+	2400 6200 2400 6250
 Wire Wire Line
 	2400 6200 3100 6200
@@
 IN1
 Wire Wire Line
-	1300 2400 1500 2400
+	1300 2400 1800 2400
 Text HLabel 1300 2700 0    60   Input ~ 0
 IN2
 Wire Wire Line
-	1300 2700 1500 2700
+	1300 2700 1800 2700
 $Comp
 L C-1206 C40
@@
 Wire Wire Line
 	3800 3500 3800 3250
+$Comp
+L R-0603 R?
+U 1 1 577963E5
+P 4500 3500
+AR Path="/57752301/577963E5" Ref="R?"  Part="1"
+AR Path="/5774BBA6/577963E5" Ref="R36"  Part="1"
+F 0 "R36" V 4700 3500 50  0000 C CNN
+F 1 "5k1" V 4609 3500 50  0000 C CNN
+F 2 "IPC7351-Nominal:RESC1608X50" H 4500 3500 50  0001 C CNN
+F 3 "" H 4500 3550 60  0000 C CNN
+F 4 "RES SMD 5k1 1% [0603]" H 5250 4050 60  0001 C CNN "BOM"
+	1    4500 3500
+	0    -1   -1   0
+$EndComp
+Wire Wire Line
+	4600 3500 4700 3500
+Wire Wire Line
+	4400 3500 4000 3500
+Wire Wire Line
+	4000 3500 3800 3500
+$Comp
+L SCHOTTKY-CK D3
+U 1 1 577EA45B
+P 2300 2000
+F 0 "D3" V 2346 1895 50  0000 R CNN
+F 1 "MBRD1035CTLT4G" V 2255 1895 50  0000 R CNN
+F 2 "" V 2250 2000 60  0000 C CNN
+F 3 "" V 2250 2000 60  0000 C CNN
+F 4 "DIST DIGIKEY MBRD1035CTLT4GOSCT-ND" H 2300 2000 60  0001 C CNN "BOM"
+	1    2300 2000
+	0    -1   -1   0
+$EndComp
+Text Notes 2500 1800 0    60   ~ 0
+REV2: add this diode here
+$Comp
+L R-0603 R37
+U 1 1 577EA74D
+P 3600 3300
+F 0 "R37" H 3537 3254 50  0000 R CNN
+F 1 "100k" H 3537 3345 50  0000 R CNN
+F 2 "IPC7351-Nominal:RESC1608X50" H 3600 3300 50  0001 C CNN
+F 3 "" H 3600 3350 60  0000 C CNN
+F 4 "RES SMD 100k 1% [0603]" H 4350 3850 60  0001 C CNN "BOM"
+	1    3600 3300
+	-1   0    0    1
+$EndComp
+Text Notes 2800 2850 0    60   ~ 0
+REV2: add this res here
 $EndSCHEMATC
